File: dc-motor.sch (EAGLE design)
At the start: 0 parts

Commit message: Erste Version des Schaltplans (Noch nicht fertig)
Parts:
- added C1, C10, C13, C14, C3, C9: 100nF, Capacitor:C-BELAB0805
- added C11: 1µF, Capacitor:C-BELAB0805
- added C12: 0,22µF, Capacitor:C-BELAB0805
- added C2, C7, C8: 10nF, Capacitor:C-BELAB0805
- added C4: 100µF/50V, Capacitor:ELK_STEHEND_5_13
- added C5: 47µF, Capacitor:ELK_STEHEND_5_13
- added C6: 100µF, Capacitor:ELK_STEHEND_5_13
- added D1: 1N4007, Diode:1N4007
- added D2: 1,5KB33CA, Diode:P6KEXXC
- added F1: F2A, fuse:F457
- added F2: T0,5A, fuse:F457
- added G1: 8MHz, Crystals:CRYTAL
- added H1, H2: MOUNT-PAD-ROUND3.0, Holes:MOUNT-PAD-ROUND3.0
- added IC1: MEGA8-P, atmel:MEGA8-P
- added JP1, JP2, JP3: (no value), jumper:JP2QE
- added R1: (no value), DC-DC-converter:R-785.0-0.5
- added R10, R3, R8, R9: 2k7, Resistor:0805
- added R11, R4, R6: 39k, Resistor:0805
- added R12, R5, R7: 10k, Resistor:0805
- added R13, R14, R15: 3,3k, Resistor:0805
- added R16, R17, R18, R19: 180R, Resistor:0805
- added R2: 0,05R, Resistor:SMS-0
- added R20, R21, R22, R23: 250R, Resistor:0805
- added S1: (no value), Switch:10-XX
- added S2, S3: (no value), Switch:DRUCKTASTER_ABGW
- added U$17: MAX4080, Sensorics:MAX4080
- added U$28: ACPL-247, Optoelectronic:ACPL-247
- added U$3: DRV-8800, DRV-8800:DRV-8800
- added X1: (no value), con-subd:F09HP
- added X2: (no value), con-subd:M09HP
- added X3, X4: RIA_3POL, Connector:RIA_3POL
- added X5: RIA_2POL, Connector:RIA_2POL
- added X6: JUMP1-4, Connector:JUMP1-4
Connections:
- new net +24V: C5.+, D1.K, D2.2, F1.1, F2.2, R1.1, R11.2
- new net GND: C1.1, C10.1, C12.1, C14.1, C2.1, C4.-, C5.-, C6.-, C7.1, C8.1, C9.1, D1.A, D2.1, IC1.GND, IC1.GND@1, R1.2, R10.1, R12.1, R15.2, R3.1, R5.1, R7.1, R8.1, R9.1, S1.P, S1.P1, U$17.GND, U$28G$1.C, U$28G$2.C, U$28G$3.C, U$28G$4.C, U$3.GND, U$3.GND1, X1.G1, X1.G2, X2.6, X2.7, X2.G2, X5.2.STIFT, X6.4
- new net N$1: F1.2, X2.1, X5.1.STIFT
- new net N$10: C13.1, C14.2, C4.+, R2.2, U$17.RS-, U$3.VBB
- new net N$11: IC1.PB4(MISO), R6.1, R7.2
- new net N$12: R6.2, X2.9
- new net N$13: R4.2, X2.8
- new net N$14: IC1.PC0(ADC0), U$17.OUT
- new net N$15: IC1.PB3(MOSI/OC2), R8.2, S3.C
- new net N$16: C3.1
- new net N$17: IC1.PB2(SS/OC1B), R3.2, S2.C
- new net N$18: IC1.PB1(OC1A), JP1-1.1, JP1-2.1, R9.2
- new net N$19: JP1-1.2, JP2-1.2, X1.3
- new net N$2: G1.2, IC1.PB6(XTAL1/TOSC1)
- new net N$20: JP1-2.2, JP2-2.2, X1.2
- new net N$21: H1.MOUNT
- new net N$22: IC1.PC6(/RESET), S1.S, S1.S1
- new net N$23: C8.2, IC1.AVCC
- new net N$24: C10.2, H2.MOUNT
- new net N$25: IC1.PB0(ICP), JP2-1.1, JP2-2.1, R10.2
- new net N$26: C11.2, U$3.CP1
- new net N$27: C11.1, U$3.CP2
- new net N$28: C12.2, U$3.VREG
- new net N$29: C13.2, U$3.VCP
- new net N$3: G1.1, IC1.PB7(XTAL2/TOSC2)
- new net N$30: IC1.PC2(ADC2)
- new net N$31: R23.1, U$3.ENABLE
- new net N$32: R21.1, U$3.PHASE
- new net N$33: R14.1, U$3.NFAULT
- new net N$34: R13.1, R20.1, U$3.NSLEEP
- new net N$35: U$28G$1.EMIT
- new net N$36: R15.1, U$3.SENSE
- new net N$38: IC1.PD5(T1), R16.1
- new net N$39: IC1.PD4(XCK/T0), R19.1
- new net N$4: IC1.PD0(RXD), X6.1
- new net N$40: IC1.PD3(INT1), R18.2
- new net N$41: R17.2
- new net N$42: R16.2, U$28G$1.A
- new net N$43: R17.1, U$28G$2.A
- new net N$44: R18.1, U$28G$3.A
- new net N$45: R19.2, U$28G$4.A
- new net N$46: R23.2, U$28G$2.EMIT
- new net N$47: R21.2, U$28G$3.EMIT
- new net N$48: R22.1, U$3.MODE
- new net N$49: R20.2, U$28G$4.EMIT
- new net N$5: JP3-1.1, JP3-2.2, U$3.OUT+, X1.4
- new net N$50: IC1.PC1(ADC1), R11.1, R12.2
- new net N$51: IC1.PC3(ADC3)
- new net N$52: IC1.PC4(ADC4/SDA)
- new net N$53: IC1.PC5(ADC5/SCL)
- new net N$6: F2.1, R2.1, U$17.RS+
- new net N$7: JP3-1.2, JP3-2.1, U$3.OUT-, X1.5
- new net N$8: IC1.PD1(TXD), X6.2
- new net N$9: IC1.PB5(SCK), R4.1, R5.2
- new net VDD: C1.2, C2.2, C3.2, C6.+, C7.2, IC1.AREF, IC1.VCC@1, R1.3, R13.2, R14.2, S2.N0, S3.N0, U$17.VCC, U$28G$1.COL, U$28G$2.COL, U$28G$3.COL, U$28G$4.COL, X1.1, X6.3
Other:
- note added: "ENDSCHALTER UMPOLUNG"
- note added: "PC Eingang A"
- note added: "PC Eingang B"
- note added: "TASTER A"
- note added: "TASTER B"
- note added: "UART"
