File: dc-motor.brd (EAGLE design)
At the start: 160 x 100 mm, 85 parts, among them IC1 MEGA32-A, X10 JUMP1-4, X11 JUMP1-4, X3 RIA_3POL, X4 RIA_3POL, X5 RIA_2POL, X6 JUMP1-4, X7 PFVERB10, X8 PFVERB10, X9 JUMP1-4

Commit message: Layout finished
Parts:
- removed X10, X11, X9: JUMP1-4, Connector:JUMP1-4
- moved R36 159.6 mm to (144.1, 43.2), turned to 180 degrees
- moved U$50 146.0 mm to (135.9, 41.9), turned to 270 degrees
- moved R37 140.6 mm to (128.9, 41.3), turned to 180 degrees
- moved R32 67.5 mm to (135.3, 82.5), turned to 90 degrees
- moved R31 61.5 mm to (134.0, 73.7), turned to 270 degrees
- moved C15 55.0 mm to (41.9, 43.0), turned to 180 degrees
- moved C1 48.0 mm to (57.1, 17.1), turned to 0 degrees
- moved C16 46.5 mm to (41.9, 48.1)
- moved R39 45.4 mm to (27.3, 8.26), turned to 180 degrees
- moved G1 44.5 mm to (47.6, 45.6), turned to 90 degrees
- moved R23 41.9 mm to (138.1, 6.03), turned to 270 degrees
- moved R11 41.7 mm to (96.5, 52.7), turned to 0 degrees
- moved R22 40.8 mm to (123.8, 10.8), turned to 270 degrees
- moved R12 40.8 mm to (97.8, 56.2)
- moved R13 40.0 mm to (137.8, 9.53), turned to 90 degrees
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Connections:
- removed net N$30: U$3.10, X1.5, X11.2, X11.3
- removed net N$5: U$3.7, X1.4, X11.1, X11.4
- new net +24V_LED_µC: IC1.20, X7.3
- new net MOTOR: IC1.12, X1.6
- new net N$41: U$3.7, X1.4
- new net N$44: U$3.10, X1.5
- new net RICHTUNG: IC1.11, X1.9
- net +24V: no longer X7.3
- net GND: now also X1.7, X1.8, X2.G1
- net N$18: no longer X10.1, X10.3
- net N$20: no longer X10.4, X9.4
- net N$22: no longer X10.2, X9.2
- net N$25: no longer X9.1, X9.3
- net N$39: now also U$50.7, U$50.8
- net N$60: now also IC1.29; no longer IC1.27
- net VDD: now also IC1.27; no longer IC1.29
Routing:
- net N$6: track 15.6 -> 236.0 mm, vias 0 -> 2
- net VDD: track 319.4 -> 529.6 mm, vias 1 -> 5
- net +24V: track 124.7 -> 318.6 mm, vias 0 -> 1
- net SCK: track 3.15 -> 196.7 mm, vias 0 -> 3
- net MISO: track 3.74 -> 186.7 mm, vias 0 -> 3
- net MOSI: track 3.91 -> 180.4 mm, vias 0 -> 1
- net VOLTAGE_FUSE: track 0.00 -> 169.0 mm, vias 0 -> 2
- net N$15: track 8.81 -> 160.0 mm, vias 1 -> 2
- net N$17: track 2.43 -> 152.3 mm, vias 0 -> 4
- net N$38: track 3.91 -> 153.7 mm, vias 0 -> 2
- net LOCAL/REMOTE: track 3.28 -> 141.8 mm, vias 0 -> 3
- net ENDLAGE_A: track 11.1 -> 140.6 mm, vias 0 -> 2
- net N$22: track 37.8 -> 159.9 mm
- net RICHTUNG: track 0.00 -> 121.3 mm, vias 0 -> 1
- net ENDLAGE_B: track 15.4 -> 134.9 mm
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
Commit message: layout checked
Parts:
- moved H1 2.05 mm to (3.13, 94.6)
- moved R15 1.78 mm to (142.2, 16.6)
- moved C10 0.63 mm to (15.2, 5.08)
- moved C5 0.63 mm to (41.9, 8.89)
- moved C9 0.63 mm to (15.0, 94.7)
- moved H2 0.43 mm to (3.10, 5.29)
Connections:
- net MOTORSICHERUNGLED renamed FEHLER_LED
- removed net N$20: X1.2, X7.2
- removed net N$22: X1.3, X7.1
- net N$18: now also X1.3, X7.1
- net N$25: now also X1.2, X7.2
Routing:
- net N$18: track 19.4 -> 214.2 mm, vias 0 -> 3
- net N$25: track 18.9 -> 202.4 mm, vias 0 -> 3
- net N$20: track 161.8 -> 0.00 mm
- net N$22: track 159.9 -> 0.00 mm
- net N$6: track 236.0 -> 228.7 mm, vias 2 -> 1
- net N$41: track 16.8 -> 11.8 mm
- net N$36: track 5.74 -> 3.88 mm
- net N$21: track 9.21 -> 11.0 mm
- net VDD: track 529.6 -> 530.9 mm
- net N$16: track 75.9 -> 74.7 mm
- net N$9: track 78.4 -> 79.3 mm
- net LOCAL/REMOTE: track 141.8 -> 141.2 mm
- net N$8: track 75.8 -> 76.3 mm
- net N$17: track 152.3 -> 152.9 mm
