File: dc-motor.brd (EAGLE design)
At the start: 160 x 100 mm, 82 parts, among them IC1 MEGA32-A, X3 RIA_3POL, X4 RIA_3POL, X5 RIA_2POL, X6 JUMP1-4, X7 PFVERB10, X8 PFVERB10

Commit message: Layout edited
Parts:
- removed X7: PFVERB10, Connector:PFVERB10
- added SV1: (no value), con-lstb:MA06-2
- moved R3 4.44 mm to (17.8, 76.8)
- moved S2 3.81 mm to (5.08, 73.7)
- moved R10 0.32 mm to (97.5, 47.6)
- moved R9 0.32 mm to (97.5, 45.7)
Connections:
- removed net FEHLER_LED: IC1.37, X7.4
- removed net N$18: IC1.25, R9.2, X1.3, X7.1
- removed net N$25: IC1.26, R10.2, X1.2, X7.2
- new net ENDSCHALTER_A: IC1.25, R9.2, SV1.3, X1.3
- new net ENDSCHALTER_B: IC1.26, R10.2, SV1.7, X1.2
- new net RGB_BLAU: IC1.15, SV1.6
- new net RGB_GRUEN: IC1.14, SV1.2
- new net RGB_ROT: IC1.16, SV1.4
- net +24V_LED_µC: now also SV1.8; no longer IC1.20, X7.3
- net FAEHRTNACHA: now also SV1.1; no longer X7.5
- net FAEHRTNACHB: now also SV1.5; no longer X7.6
- net GND: now also SV1.11; no longer X7.10
- net LOCAL/REMOTE: now also SV1.10; no longer X7.8
- net MOTORSTOP: now also SV1.9; no longer X7.7
- net NFAULT: now also IC1.20; no longer IC1.19
- net VDD: now also SV1.12; no longer X7.9
Routing:
- net N$18: track 214.2 -> 0.00 mm, vias 3 -> 0
- net ENDSCHALTER_B: track 0.00 -> 205.2 mm, vias 0 -> 5
- net ENDSCHALTER_A: track 0.00 -> 203.5 mm, vias 0 -> 3
- net N$25: track 202.4 -> 0.00 mm, vias 3 -> 0
- net +24V_LED_µC: track 84.6 -> 0.00 mm, vias 1 -> 0
- net RGB_BLAU: track 0.00 -> 83.4 mm, vias 0 -> 3
- net RGB_ROT: track 0.00 -> 77.0 mm, vias 0 -> 3
- net RGB_GRUEN: track 0.00 -> 67.2 mm, vias 0 -> 3
- net FEHLER_LED: track 59.3 -> 0.00 mm, vias 1 -> 0
- net LOCAL/REMOTE: track 141.2 -> 151.0 mm, vias 3 -> 5
- net MOTORSTOP: track 63.1 -> 71.5 mm
- net FAEHRTNACHB: track 71.1 -> 62.9 mm
- net VDD: track 530.9 -> 527.1 mm
- net VOLTAGE_FUSE: track 169.2 -> 167.8 mm
- net FAEHRTNACHA: track 57.9 -> 59.1 mm
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
Commit message: edited again
Parts:
- moved R10 31.4 mm to (69.2, 34.0), turned to 90 degrees
- moved R9 2.62 mm to (98.1, 48.3)
Connections:
- net ENDSCHALTER_A: now also IC1.11; no longer IC1.25
- net ENDSCHALTER_B: now also IC1.12; no longer IC1.26
- net MOTOR: now also IC1.26; no longer IC1.12
- net RICHTUNG: now also IC1.25; no longer IC1.11
Routing:
- net ENDSCHALTER_B: track 205.2 -> 186.0 mm, vias 5 -> 3
- net RICHTUNG: track 121.8 -> 107.6 mm, vias 1 -> 3
- net ENDSCHALTER_A: track 203.5 -> 209.1 mm, vias 3 -> 6
- net MOTOR: track 102.9 -> 98.5 mm
- net N$17: track 153.8 -> 152.8 mm
- net RGB_BLAU: track 83.4 -> 84.1 mm, vias 3 -> 1
- net RGB_ROT: vias 3 -> 1
- net RGB_GRUEN: vias 3 -> 1
